File: foArduinoMega.brd (EAGLE design)
At the start: 47 x 72 mm, 14 parts

Commit message: #release Adafruit ciruit
Parts:
- renumbered CN1 to BALL1, CN11 to PING4, CN12 to PING3, CN13 to PING2, CN14 to PING1, CN2 to BALL2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
